File: layouts/particle-counter/particle-counter.kicad_pcb (KiCad board)
At the start: 2 copper layers, 22 parts

Commit message: changed main target to mainboard, added cutoff build, lots of edits to modules
Connections:
- C3 pad 2: net-1 -> net
- C7 pad 1: net -> unnamed[1]
- C8 pad 1: net -> unnamed[1]
- R4 pad 1: net-1 -> net
- R8 pad 2: net -> unnamed[1]

Commit message: finished cutoff mechanism connections :fixed
Connections:
- C2 pad 1: C3-net-1 -> C3-net
- C2 pad 2: C3-net -> C3-net-1
- C3 pad 2: net -> net-1
- C7 pad 1: unnamed[1] -> net
- C8 pad 1: unnamed[1] -> net
- R4 pad 1: net -> net-1
- R8 pad 2: unnamed[1] -> net
Changed lines of the file:
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@@
     (net 1 "VCC")
     (net 2 "OUT1")
-    (net 3 "C3-net")
+    (net 3 "C3-net-1")
     (net 4 "IN2plus")
     (net 5 "IN1plus")
-    (net 6 "net")
-    (net 7 "C3-net-1")
+    (net 6 "net-1")
+    (net 7 "C3-net")
     (net 8 "IN2minus")
     (net 9 "K")
     (net 10 "gnd")
-    (net 11 "unnamed[1]")
+    (net 11 "net")
     (net 12 "OUTPUT")
     (net 13 "OUT2")
@@
             (size 0.79 0.54)
             (layers "F.Cu" "F.Mask" "F.Paste")
-            (net 6 "net")
+            (net 6 "net-1")
         )
         (embedded_fonts no)
@@
             (size 0.79 0.54)
             (layers "F.Cu" "F.Mask" "F.Paste")
-            (net 11 "unnamed[1]")
+            (net 11 "net")
         )
         (pad "2" smd rect
@@
             (size 0.79 0.54)
             (layers "F.Cu" "F.Mask" "F.Paste")
-            (net 7 "C3-net-1")
+            (net 7 "C3-net")
         )
         (pad "2" smd rect
@@
             (size 0.79 0.54)
             (layers "F.Cu" "F.Mask" "F.Paste")
-            (net 3 "C3-net")
+            (net 3 "C3-net-1")
         )
         (embedded_fonts no)
@@
             (size 0.3 0.32)
             (layers "F.Cu" "F.Mask" "F.Paste")
-            (net 6 "net")
+            (net 6 "net-1")
         )
         (pad "2" smd rect
@@
             (size 0.79 0.54)
             (layers "F.Cu" "F.Mask" "F.Paste")
-            (net 11 "unnamed[1]")
+            (net 11 "net")
         )
         (pad "2" smd rect
@@
             (size 0.81 0.86)
             (layers "F.Cu" "F.Mask" "F.Paste")
-            (net 11 "unnamed[1]")
+            (net 11 "net")
         )
         (embedded_fonts no)

Commit message: major updates
Connections:
- net OUTPUT renamed out
- C2 pad 1: C3-net -> C3-net-1
- C2 pad 2: C3-net-1 -> C3-net
- C3 pad 2: net-1 -> net
- C7 pad 1: net -> net-1
- C8 pad 1: net -> net-1
- R4 pad 1: net-1 -> net
- R8 pad 2: net -> net-1
Changed lines of the file:
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@@
     (net 1 "VCC")
     (net 2 "OUT1")
-    (net 3 "C3-net-1")
+    (net 3 "C3-net")
     (net 4 "IN2plus")
     (net 5 "IN1plus")
-    (net 6 "net-1")
-    (net 7 "C3-net")
+    (net 6 "net")
+    (net 7 "C3-net-1")
     (net 8 "IN2minus")
     (net 9 "K")
     (net 10 "gnd")
-    (net 11 "net")
-    (net 12 "OUTPUT")
+    (net 11 "net-1")
+    (net 12 "out")
     (net 13 "OUT2")
     (footprint "atopile:C0402-b3ef17"
@@
             (size 0.79 0.54)
             (layers "F.Cu" "F.Mask" "F.Paste")
-            (net 6 "net-1")
+            (net 6 "net")
         )
         (embedded_fonts no)
@@
             (size 0.79 0.54)
             (layers "F.Cu" "F.Mask" "F.Paste")
-            (net 11 "net")
+            (net 11 "net-1")
         )
         (pad "2" smd rect
@@
             (size 0.79 0.54)
             (layers "F.Cu" "F.Mask" "F.Paste")
-            (net 12 "OUTPUT")
+            (net 12 "out")
         )
         (embedded_fonts no)
@@
             (size 0.79 0.54)
             (layers "F.Cu" "F.Mask" "F.Paste")
-            (net 7 "C3-net")
+            (net 7 "C3-net-1")
         )
         (pad "2" smd rect
@@
             (size 0.79 0.54)
             (layers "F.Cu" "F.Mask" "F.Paste")
-            (net 3 "C3-net-1")
+            (net 3 "C3-net")
         )
         (embedded_fonts no)
@@
             (size 0.3 0.32)
             (layers "F.Cu" "F.Mask" "F.Paste")
-            (net 6 "net-1")
+            (net 6 "net")
         )
         (pad "2" smd rect
@@
             (size 0.3 0.32)
             (layers "F.Cu" "F.Mask" "F.Paste")
-            (net 12 "OUTPUT")
+            (net 12 "out")
         )
         (pad "2" smd rect
@@
             (size 0.79 0.54)
             (layers "F.Cu" "F.Mask" "F.Paste")
-            (net 11 "net")
+            (net 11 "net-1")
         )
         (pad "2" smd rect
@@
             (size 0.81 0.86)
             (layers "F.Cu" "F.Mask" "F.Paste")
-            (net 11 "net")
+            (net 11 "net-1")
         )
         (embedded_fonts no)

Commit message: added boost buck
Connections:
- C2 pad 1: C3-net-1 -> C3-net
- C2 pad 2: C3-net -> C3-net-1
- C3 pad 2: net -> net-1
- C7 pad 1: net-1 -> net
- C8 pad 1: net-1 -> net
- R4 pad 1: net -> net-1
- R8 pad 2: net-1 -> net
Changed lines of the file:
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@@
     (net 1 "VCC")
     (net 2 "OUT1")
-    (net 3 "C3-net")
+    (net 3 "C3-net-1")
     (net 4 "IN2plus")
     (net 5 "IN1plus")
-    (net 6 "net")
-    (net 7 "C3-net-1")
+    (net 6 "net-1")
+    (net 7 "C3-net")
     (net 8 "IN2minus")
     (net 9 "K")
     (net 10 "gnd")
-    (net 11 "net-1")
+    (net 11 "net")
     (net 12 "out")
     (net 13 "OUT2")
@@
             (size 0.79 0.54)
             (layers "F.Cu" "F.Mask" "F.Paste")
-            (net 6 "net")
+            (net 6 "net-1")
         )
         (embedded_fonts no)
@@
             (size 0.79 0.54)
             (layers "F.Cu" "F.Mask" "F.Paste")
-            (net 11 "net-1")
+            (net 11 "net")
         )
         (pad "2" smd rect
@@
             (size 0.79 0.54)
             (layers "F.Cu" "F.Mask" "F.Paste")
-            (net 7 "C3-net-1")
+            (net 7 "C3-net")
         )
         (pad "2" smd rect
@@
             (size 0.79 0.54)
             (layers "F.Cu" "F.Mask" "F.Paste")
-            (net 3 "C3-net")
+            (net 3 "C3-net-1")
         )
         (embedded_fonts no)
@@
             (size 0.3 0.32)
             (layers "F.Cu" "F.Mask" "F.Paste")
-            (net 6 "net")
+            (net 6 "net-1")
         )
         (pad "2" smd rect
@@
             (size 0.79 0.54)
             (layers "F.Cu" "F.Mask" "F.Paste")
-            (net 11 "net-1")
+            (net 11 "net")
         )
         (pad "2" smd rect
@@
             (size 0.81 0.86)
             (layers "F.Cu" "F.Mask" "F.Paste")
-            (net 11 "net-1")
+            (net 11 "net")
         )
         (embedded_fonts no)

Commit message: pcb layout
Connections:
- C2 pad 1: C3-net -> C3-net-1
- C2 pad 2: C3-net-1 -> C3-net
- C3 pad 2: net-1 -> net
- C7 pad 1: net -> net-1
- C8 pad 1: net -> net-1
- R4 pad 1: net-1 -> net
- R8 pad 2: net -> net-1
Changed lines of the file:
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@@
     (net 1 "VCC")
     (net 2 "OUT1")
-    (net 3 "C3-net-1")
+    (net 3 "C3-net")
     (net 4 "IN2plus")
     (net 5 "IN1plus")
-    (net 6 "net-1")
-    (net 7 "C3-net")
+    (net 6 "net")
+    (net 7 "C3-net-1")
     (net 8 "IN2minus")
     (net 9 "K")
     (net 10 "gnd")
-    (net 11 "net")
+    (net 11 "net-1")
     (net 12 "out")
     (net 13 "OUT2")
@@
             (size 0.79 0.54)
             (layers "F.Cu" "F.Mask" "F.Paste")
-            (net 6 "net-1")
+            (net 6 "net")
         )
         (embedded_fonts no)
@@
             (size 0.79 0.54)
             (layers "F.Cu" "F.Mask" "F.Paste")
-            (net 11 "net")
+            (net 11 "net-1")
         )
         (pad "2" smd rect
@@
             (size 0.79 0.54)
             (layers "F.Cu" "F.Mask" "F.Paste")
-            (net 7 "C3-net")
+            (net 7 "C3-net-1")
         )
         (pad "2" smd rect
@@
             (size 0.79 0.54)
             (layers "F.Cu" "F.Mask" "F.Paste")
-            (net 3 "C3-net-1")
+            (net 3 "C3-net")
         )
         (embedded_fonts no)
@@
             (size 0.3 0.32)
             (layers "F.Cu" "F.Mask" "F.Paste")
-            (net 6 "net-1")
+            (net 6 "net")
         )
         (pad "2" smd rect
@@
             (size 0.79 0.54)
             (layers "F.Cu" "F.Mask" "F.Paste")
-            (net 11 "net")
+            (net 11 "net-1")
         )
         (pad "2" smd rect
@@
             (size 0.81 0.86)
             (layers "F.Cu" "F.Mask" "F.Paste")
-            (net 11 "net")
+            (net 11 "net-1")
         )
         (embedded_fonts no)
