File: layouts/cutoff/cutoff.kicad_pcb (KiCad board)
At the start: 2 copper layers, 4 parts

Commit message: major updates
Parts:
- added D1: , atopile:SMA_L4.3-W2.6-LS5.2-RD-e14692, F.Cu at (0.00, -10.0)
- added Q2: , atopile:TO-220-3_L10.0-W4.5-P2.54-L-8dee21, F.Cu at (0.00, -20.0)
- added R2: 10kΩ ±1% 62.5mW, atopile:R0402-56259e, F.Cu at (0.00, 0.00)
- added R3: 10kΩ ±1% 62.5mW, atopile:R0402-56259e, F.Cu at (0.00, -20.0)
- added R4: 10kΩ ±1% 62.5mW, atopile:R0402-56259e, F.Cu at (0.00, -10.0)
- R1: value 1kΩ ±1% 62.5mW -> 10kΩ ±1% 62.5mW
- moved Q1 20.0 mm to (0.00, 0.00)
Connections:
- net GATE renamed SC_GATE
- net unnamed[1] renamed K
- C1 pad 2: gnd -> C-1
- Q1 pad 2: C -> C-1

Commit message: added boost buck
Connections:
- C1 pad 2: C-1 -> C
- P1 pad 2: C -> C-1
- Q1 pad 2: C-1 -> C
- Q2 pad 2: C -> C-1
Changed lines of the file:
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@@
     (net 2 "hv")
     (net 7 "SC_GATE")
-    (net 10 "C-1")
-    (net 11 "C")
+    (net 10 "C")
+    (net 11 "C-1")
     (net 1 "K")
     (net 3 "SC_Sense")
@@
             (drill oval 1.9999959999999999 1.199896)
             (layers "*.Cu" "*.Mask")
-            (net 11 "C")
+            (net 11 "C-1")
         )
     )
@@
             (drill 0.9999979999999999)
             (layers "*.Cu" "*.Mask")
-            (net 10 "C-1")
+            (net 10 "C")
         )
         (pad "1" thru_hole circle
@@
             (drill 1.1999975999999999)
             (layers "*.Cu" "*.Mask")
-            (net 10 "C-1")
+            (net 10 "C")
         )
         (pad "3" thru_hole oval
@@
             (drill 1.1999975999999999)
             (layers "*.Cu" "*.Mask")
-            (net 11 "C")
+            (net 11 "C-1")
         )
         (pad "3" thru_hole oval

Commit message: built
Parts:
- R1, R2, R3, R4: value 10kΩ ±1% 62.5mW -> 1kΩ ±1% 62.5mW
Changed lines of the file:
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@@
             )
         )
-        (property "Value" "10kΩ ±1% 62.5mW"
+        (property "Value" "1kΩ ±1% 62.5mW"
             (at 0 4 0)
             (layer "F.Fab")
@@
             )
         )
-        (property "LCSC" "C25744"
-            (at 0 0 0)
-            (layer "User.9")
-            (hide yes)
-            (effects
-                (font
-                    (size 0.125 0.125)
-                    (thickness 0.01875)
-                )
-            )
-        )
-        (property "Partnumber" "0402WGF1002TCE"
+        (property "LCSC" "C11702"
+            (at 0 0 0)
+            (layer "User.9")
+            (hide yes)
+            (effects
+                (font
+                    (size 0.125 0.125)
+                    (thickness 0.01875)
+                )
+            )
+        )
+        (property "Partnumber" "0402WGF1001TCE"
             (at 0 0 0)
             (layer "User.9")
@@
             )
         )
-        (property "JLCPCB description" "62.5mW Thick Film Resistors 50V ±100ppm/℃ ±1% 10kΩ 0402 Chip Resistor - Surface Mount ROHS"
+        (property "JLCPCB description" "62.5mW Thick Film Resistors 50V ±100ppm/℃ ±1% 1kΩ 0402 Chip Resistor - Surface Mount ROHS"
             (at 0 0 0)
             (layer "User.9")
@@
             )
         )
-        (property "PARAM_resistance" "{\"type\": \"Quantity_Interval_Disjoint\", \"data\": {\"intervals\": {\"type\": \"Numeric_Interval_Disjoint\", \"data\": {\"intervals\": [{\"type\": \"Numeric_Interval\", \"data\": {\"min\": 9900.000002235174, \"max\": 10099.999997764826}}]}}, \"unit\": \"ohm\"}}"
+        (property "PARAM_resistance" "{\"type\": \"Quantity_Interval_Disjoint\", \"data\": {\"intervals\": {\"type\": \"Numeric_Interval_Disjoint\", \"data\": {\"intervals\": [{\"type\": \"Numeric_Interval\", \"data\": {\"min\": 990.0000002235174, \"max\": 1009.9999997764826}}]}}, \"unit\": \"ohm\"}}"
             (at 0 0 0)
             (layer "User.9")
@@
             )
         )
-        (property "Value" "10kΩ ±1% 62.5mW"
+        (property "Value" "1kΩ ±1% 62.5mW"
             (at 0 4 0)
             (layer "F.Fab")
@@
             )
         )
-        (property "LCSC" "C25744"
-            (at 0 0 0)
-            (layer "User.9")
-            (hide yes)
-            (effects
-                (font
-                    (size 0.125 0.125)
-                    (thickness 0.01875)
-                )
-            )
-        )
-        (property "Partnumber" "0402WGF1002TCE"
+        (property "LCSC" "C11702"
+            (at 0 0 0)
+            (layer "User.9")
+            (hide yes)
+            (effects
+                (font
+                    (size 0.125 0.125)
+                    (thickness 0.01875)
+                )
+            )
+        )
+        (property "Partnumber" "0402WGF1001TCE"
             (at 0 0 0)
             (layer "User.9")
@@
             )
         )
-        (property "JLCPCB description" "62.5mW Thick Film Resistors 50V ±100ppm/℃ ±1% 10kΩ 0402 Chip Resistor - Surface Mount ROHS"
+        (property "JLCPCB description" "62.5mW Thick Film Resistors 50V ±100ppm/℃ ±1% 1kΩ 0402 Chip Resistor - Surface Mount ROHS"
             (at 0 0 0)
             (layer "User.9")
@@
             )
         )
-        (property "PARAM_resistance" "{\"type\": \"Quantity_Interval_Disjoint\", \"data\": {\"intervals\": {\"type\": \"Numeric_Interval_Disjoint\", \"data\": {\"intervals\": [{\"type\": \"Numeric_Interval\", \"data\": {\"min\": 9900.000002235174, \"max\": 10099.999997764826}}]}}, \"unit\": \"ohm\"}}"
+        (property "PARAM_resistance" "{\"type\": \"Quantity_Interval_Disjoint\", \"data\": {\"intervals\": {\"type\": \"Numeric_Interval_Disjoint\", \"data\": {\"intervals\": [{\"type\": \"Numeric_Interval\", \"data\": {\"min\": 990.0000002235174, \"max\": 1009.9999997764826}}]}}, \"unit\": \"ohm\"}}"
             (at 0 0 0)
             (layer "User.9")
@@
             )
         )
-        (property "Value" "10kΩ ±1% 62.5mW"
+        (property "Value" "1kΩ ±1% 62.5mW"
             (at 0 4 0)
             (layer "F.Fab")
@@
             )
         )
-        (property "LCSC" "C25744"
-            (at 0 0 0)
-            (layer "User.9")
-            (hide yes)
-            (effects
-                (font
-                    (size 0.125 0.125)
-                    (thickness 0.01875)
-                )
-            )
-        )
-        (property "Partnumber" "0402WGF1002TCE"
+        (property "LCSC" "C11702"
+            (at 0 0 0)
+            (layer "User.9")
+            (hide yes)
+            (effects
+                (font
+                    (size 0.125 0.125)
+                    (thickness 0.01875)
+                )
+            )
+        )
+        (property "Partnumber" "0402WGF1001TCE"
             (at 0 0 0)
             (layer "User.9")
@@
             )
         )
-        (property "JLCPCB description" "62.5mW Thick Film Resistors 50V ±100ppm/℃ ±1% 10kΩ 0402 Chip Resistor - Surface Mount ROHS"
+        (property "JLCPCB description" "62.5mW Thick Film Resistors 50V ±100ppm/℃ ±1% 1kΩ 0402 Chip Resistor - Surface Mount ROHS"
             (at 0 0 0)
             (layer "User.9")
@@
             )
         )
-        (property "PARAM_resistance" "{\"type\": \"Quantity_Interval_Disjoint\", \"data\": {\"intervals\": {\"type\": \"Numeric_Interval_Disjoint\", \"data\": {\"intervals\": [{\"type\": \"Numeric_Interval\", \"data\": {\"min\": 9900.000002235174, \"max\": 10099.999997764826}}]}}, \"unit\": \"ohm\"}}"
+        (property "PARAM_resistance" "{\"type\": \"Quantity_Interval_Disjoint\", \"data\": {\"intervals\": {\"type\": \"Numeric_Interval_Disjoint\", \"data\": {\"intervals\": [{\"type\": \"Numeric_Interval\", \"data\": {\"min\": 990.0000002235174, \"max\": 1009.9999997764826}}]}}, \"unit\": \"ohm\"}}"
             (at 0 0 0)
             (layer "User.9")
@@
             )
         )
-        (property "Value" "10kΩ ±1% 62.5mW"
+        (property "Value" "1kΩ ±1% 62.5mW"
             (at 0 4 0)
             (layer "F.Fab")
@@
             )
         )
-        (property "LCSC" "C25744"
-            (at 0 0 0)
-            (layer "User.9")
-            (hide yes)
-            (effects
-                (font
-                    (size 0.125 0.125)
-                    (thickness 0.01875)
-                )
-            )
-        )
-        (property "Partnumber" "0402WGF1002TCE"
+        (property "LCSC" "C11702"
+            (at 0 0 0)
+            (layer "User.9")
+            (hide yes)
+            (effects
+                (font
+                    (size 0.125 0.125)
+                    (thickness 0.01875)
+                )
+            )
+        )
+        (property "Partnumber" "0402WGF1001TCE"
             (at 0 0 0)
             (layer "User.9")
@@
             )
         )
-        (property "JLCPCB description" "62.5mW Thick Film Resistors 50V ±100ppm/℃ ±1% 10kΩ 0402 Chip Resistor - Surface Mount ROHS"
+        (property "JLCPCB description" "62.5mW Thick Film Resistors 50V ±100ppm/℃ ±1% 1kΩ 0402 Chip Resistor - Surface Mount ROHS"
             (at 0 0 0)
             (layer "User.9")
@@
             )
         )
-        (property "PARAM_resistance" "{\"type\": \"Quantity_Interval_Disjoint\", \"data\": {\"intervals\": {\"type\": \"Numeric_Interval_Disjoint\", \"data\": {\"intervals\": [{\"type\": \"Numeric_Interval\", \"data\": {\"min\": 9900.000002235174, \"max\": 10099.999997764826}}]}}, \"unit\": \"ohm\"}}"
-            (at 0 0 0)
-            (layer "User.9")
+        (property "PARAM_resistance" "{\"type\": \"Quantity_Interval_Disjoint\", \"data\": {\"intervals\": {\"type\": \"Numeric_Interval_Disjoint\", \"data\": {\"intervals\": [{\"type\": \"Numeric_Interval\", \"data\": {\"min\": 990.0000002235174, \"max\": 1009.9999997764826}}]}}, \"unit\": \"ohm\"}}"
+            (at 0 0 0)
+            (layer "User.9")

Commit message: layout updates
Parts:
- P1: footprint atopile:CONN-TH_2P-P9.50_WJ45C-B-2P-7aea0b -> atopile:CONN-TH_2P-P5.00_WJ128V-5.0-2P-75f14f
Connections:
- C1 pad 2: C -> C-1
- P1 pad 2: C-1 -> C
- Q1 pad 2: C -> C-1
- Q2 pad 2: C-1 -> C

Commit message: added new oled
Parts:
- Q1: footprint atopile:TO-220-3_L10.0-W4.5-P2.54-L-8dee21 -> atopile:SOT-23-3_L2.9-W1.3-P1.90-LS2.4-BR-688f29
- Q2: footprint atopile:TO-220-3_L10.0-W4.5-P2.54-L-8dee21 -> atopile:DFN-8_L3.3-W3.3-P0.65-BL-2-bd6bc9
Connections:
- Q1 pad 2: C-1 -> gnd
- Q1 pad 3: gnd -> C-1
- Q2 pad 1: CUTOFF_GATE -> gnd
- Q2 pad 2: C -> gnd

Commit message: desktop push
Connections:
- C1 pad 2: C-1 -> C
- P1 pad 2: C -> C-1
- Q1 pad 3: C-1 -> C
- Q2 pad 5: C -> C-1
Changed lines of the file:
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@@
     (net 1 "K")
     (net 3 "SC_Sense")
-    (net 6 "C-1")
-    (net 8 "C")
+    (net 6 "C")
+    (net 8 "C-1")
     (net 9 "gnd")
     (net 12 "CUTOFF_GATE")
@@
             (drill 1.199896)
             (layers "*.Cu" "*.Mask")
-            (net 8 "C")
+            (net 8 "C-1")
         )
     )
@@
             (drill 0.9999979999999999)
             (layers "*.Cu" "*.Mask")
-            (net 6 "C-1")
+            (net 6 "C")
         )
         (pad "1" thru_hole circle
@@
             (size 1.25 0.7)
             (layers "F.Cu" "F.Paste" "F.Mask")
-            (net 6 "C-1")
+            (net 6 "C")
         )
     )
@@
                 )
             )
-            (net 8 "C")
+            (net 8 "C-1")
         )
         (pad "1" smd rect

Commit message: im cooking
Parts:
- removed P1: , atopile:CONN-TH_2P-P5.00_WJ128V-5.0-2P-75f14f
- added CN1: , atopile:CONN-TH_XH-2A-b4a6f6, F.Cu at (0.00, 0.00)
- added CN2: , atopile:CONN-TH_XH-2A-b4a6f6, F.Cu at (0.00, -30.0)
- added Q3: , atopile:SOT-23-3_L2.9-W1.3-P1.90-LS2.4-BR-688f29, F.Cu at (0.00, -20.0)
- R1, R2, R3, R4: value 1kΩ ±1% 62.5mW -> 10kΩ ±1% 62.5mW
- moved Q2 10.0 mm to (0.00, -10.0)
Connections:
- net C renamed C-2

Commit message: im cooking
Parts:
- R1: value 10kΩ ±1% 62.5mW -> 10kΩ ±1% 125mW; footprint atopile:R0402-56259e -> atopile:R0805-c79e8b
- R2, R3, R4: value 10kΩ ±1% 62.5mW -> 1kΩ ±1% 62.5mW
Connections:
- CN1 pad 2: C-1 -> C
- CN2 pad 2: C -> C-1
- Q2 pad 5: C-1 -> C
- Q3 pad 3: C -> C-1
