File: layouts/cutoff/cutoff.kicad_pcb (KiCad board)
At the start: 2 copper layers, 11 parts

Commit message: updates
Connections:
- C1 pad 2: C-2 -> C-1
- CN2 pad 2: C-1 -> C-2
- Q1 pad 3: C-2 -> C-1
- Q3 pad 3: C-1 -> C-2
Changed lines of the file:
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@@
     (net 1 "SC_GATE")
     (net 8 "CUTOFF_GATE")
-    (net 10 "C-2")
+    (net 10 "C-1")
     (net 11 "C")
     (net 13 "gnd")
     (net 14 "HEATER_GATE")
-    (net 15 "C-1")
+    (net 15 "C-2")
     (footprint "atopile:R0805-c79e8b"
         (layer "F.Cu")
@@
             (drill 0.9999979999999999)
             (layers "*.Cu" "*.Mask")
-            (net 10 "C-2")
+            (net 10 "C-1")
         )
         (pad "1" thru_hole circle
@@
             (size 1.25 0.7)
             (layers "F.Cu" "F.Paste" "F.Mask")
-            (net 10 "C-2")
+            (net 10 "C-1")
         )
     )
@@
             (size 1.25 0.7)
             (layers "F.Cu" "F.Paste" "F.Mask")
-            (net 15 "C-1")
+            (net 15 "C-2")
         )
     )
@@
             (drill 1.1000231999999999)
             (layers "*.Cu" "*.Mask")
-            (net 15 "C-1")
+            (net 15 "C-2")
         )
     )
