File: layouts/default/default.kicad_pcb (KiCad board)
At the start: 4 copper layers, 37.6 x 39.4 mm, 52 parts, among them U19 5.1kΩ ±1% 62.5mW, U29 5.1kΩ ±1% 62.5mW

Commit message: edits
Routing:
- net NSS: track 21.3 -> 23.2 mm
Changed lines of the file:
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@@
+		(net 64)
+	)
+	(segment
+		(start 45.4225 50.2375)
+		(end 46.6875 50.2375)
+		(width 0.2)
+		(layer "F.Cu")
+		(net 64)
+	)
+	(segment
+		(start 46.6875 50.2375)
+		(end 46.75 50.3)
+		(width 0.2)
+		(layer "F.Cu")
 		(net 64)
 	)
@@
 	)
 	(via
-		(at 46.25 50.45)
+		(at 46.75 50.3)
 		(size 0.6)
 		(drill 0.3)
@@
 	)
 	(segment
-		(start 46.25 50.45)
-		(end 46.15 50.45)
+		(start 43.938244 67.954998)
+		(end 43.9 67.993242)
 		(width 0.2)
 		(layer "B.Cu")
@@
 	)
 	(segment
-		(start 43.938244 67.954998)
-		(end 43.9 67.993242)
+		(start 46.75 50.3)
+		(end 46.74867 50.30133)
 		(width 0.2)
 		(layer "B.Cu")
@@
 	)
 	(segment
-		(start 43.938244 67.954998)
-		(end 43.9 67.916754)
+		(start 46.4 50.3)
+		(end 43.9 52.8)
+		(width 0.2)
+		(layer "In1.Cu")
+		(net 64)
+	)
+	(segment
+		(start 46.75 50.3)
+		(end 46.4 50.3)
 		(width 0.2)
 		(layer "In1.Cu")
@@
 	(segment
 		(start 43.9 67.916754)
-		(end 43.9 52.8)
+		(end 43.938244 67.954998)
 		(width 0.2)
 		(layer "In1.Cu")
@@
 	(segment
 		(start 43.9 52.8)
-		(end 46.25 50.45)
+		(end 43.9 67.916754)
 		(width 0.2)
 		(layer "In1.Cu")
